Commit message: Full Robot

File: simulation/models/robot/robot.urdf.xacro (robot description, xacro)
@@ -1,4 +1,5 @@
 <?xml version='1.0'?>
 <robot name='my_robot' xmlns:xacro="http://www.ros.org/wiki/xacro">
+    <xacro:include filename="$(find simulation)/models/robot/robot.gazebo.xacro" />
     <link name='chassi'>
         <inertial>
@@ -10,5 +11,5 @@
             <origin rpy="0 0 0" xyz="0 0 0"/>
             <geometry>
-                <box size="0.4 0.2 0.1"/>
+                <box size='0.4 0.2 0.1'/>
             </geometry>
         </collision>
@@ -16,5 +17,5 @@
             <origin rpy="0 0 0" xyz="0 0 0"/>
             <geometry>
-                <box size="0.4 0.2 0.1"/>
+                <box size='0.4 0.2 0.1'/>
             </geometry>
         </visual>
@@ -22,12 +23,12 @@
     <link name='caster'>
         <inertial>
-            <mass value="0.1"/>
+            <mass value="0.5"/>
             <origin rpy="0 0 0" xyz="0 0 0"/>
             <inertia ixx="1" ixy="0.0" ixz="0.0" iyy="1" iyz="0.0" izz="1"/>
         </inertial>
-        <collision name='collision_caster'>
+        <collision name= 'collision_caster'>
             <origin rpy="0 0 0" xyz="0 0 0"/>
             <geometry>
-                <sphere radius="0.05"/>
+                <sphere radius='0.05'/>
             </geometry>
         </collision>
@@ -35,5 +36,5 @@
             <origin rpy="0 0 0" xyz="0 0 0"/>
             <geometry>
-                <sphere radius="0.05"/>
+                <sphere radius='0.05'/>
             </geometry>
         </visual>
@@ -45,5 +46,5 @@
             <inertia ixx="1" ixy="0.0" ixz="0.0" iyy="1" iyz="0.0" izz="1"/>
         </inertial>
-        <collision name='collision_left_wheel'>
+        <collision name= 'collision_left_wheel'>
             <origin rpy="0 0 0" xyz="0 0 0"/>
             <geometry>
@@ -64,5 +65,5 @@
             <inertia ixx="1" ixy="0.0" ixz="0.0" iyy="1" iyz="0.0" izz="1"/>
         </inertial>
-        <collision name='collision_left_wheel'>
+        <collision name= 'collision_right_wheel'>
             <origin rpy="0 0 0" xyz="0 0 0"/>
             <geometry>
@@ -70,5 +71,5 @@
             </geometry>
         </collision>
-        <visual name='visual_left_wheel'>
+        <visual name='visual_right_wheel'>
             <origin rpy="0 0 0" xyz="0 0 0"/>
             <geometry>
@@ -77,5 +78,43 @@
         </visual>
     </link>
-<!-- ====================Joints=================== -->
+    <link name='camera1'>
+        <inertial>
+            <mass value="0.01"/>
+            <origin rpy="0 0 0" xyz="0 0 0"/>
+            <inertia ixx="1" ixy="0.0" ixz="0.0" iyy="1" iyz="0.0" izz="1"/>
+        </inertial>
+        <collision name= 'collision_camera1'>
+            <origin rpy="0 0 0" xyz="0 0 0"/>
+            <geometry>
+                <box size='0.05 0.05 0.05'/>
+            </geometry>
+        </collision>
+        <visual name='visual_camera1'>
+            <origin rpy="0 0 0" xyz="0 0 0"/>
+            <geometry>
+                <box size='0.05 0.05 0.05'/>
+            </geometry>
+        </visual>
+    </link>
+    <link name='laser1'>
+        <inertial>
+            <mass value="0.01"/>
+            <origin rpy="0 0 0" xyz="0 0 0"/>
+            <inertia ixx="1" ixy="0.0" ixz="0.0" iyy="1" iyz="0.0" izz="1"/>
+        </inertial>
+        <collision name= 'collision_laser1'>
+            <origin rpy="0 0 0" xyz="0 0 0"/>
+            <geometry>
+                <box size='0.05 0.05 0.05'/>
+            </geometry>
+        </collision>
+        <visual name='visual_laser1'>
+            <origin rpy="0 0 0" xyz="0 0 0"/>
+            <geometry>
+                <box size='0.05 0.05 0.05'/>
+            </geometry>
+        </visual>
+    </link>
+<!--==================== Joints ====================-->
     <joint name="joint_caster" type="fixed">
         <parent link="chassi"/>
@@ -97,3 +136,13 @@
         <limit effort="-1.0" lower="-1e+16" upper="1e+16" velocity="-1.0"/>
     </joint>
+    <joint name="joint_camera1" type="fixed">
+        <parent link="chassi"/>
+        <child link="camera1"/>
+        <origin rpy="0 0 3.1415" xyz="-0.15 0 0.075"/>
+    </joint>
+    <joint name="joint_laser1" type="fixed">
+        <parent link="chassi"/>
+        <child link="laser1"/>
+        <origin rpy="0 0 3.1415" xyz="-0.2 0 0.015"/>
+    </joint>
 </robot>
